File: docs/kicad/YATAC.kicad_pcb (KiCad board)
At the start: 2 copper layers, 203.2 x 127 mm, 108 parts, among them J1 POWER IN, J2 POWER OUT, J3 AUDIO OUT, J4 KEYBOARD, J5 SERIAL, J6 DISPLAY, J7 EXPANSION, Q1 DS1233-15, Q2 BS170, SW1 RESET, U1 27C020, U10 74F138, U11 74F157, U12 16R4, U13 74F574, U14 74F574, U15 74F163, U16 74F163, U17 74F541, U18 74F574, U19 74F257, U2 74F00, U20 74F574, U21 74F574, U22 74F541, U23 74F244, U24 74F574, U25 74F574, U26 74F574, U27 74F574, U28 AS6C4008, U29 74F574, U3 74F08, U30 74F175, U31 74F04, U32 74F00, U33 74F32, U34 74F11, U35 74F163, U36 74LS163, U37 74F541, U38 74F163, U39 74LS163, U4 74F32, U40 74F541, U41 74F163, U42 74F153, U43 74F541, U44 74F574, U45 74F299, U46 74F574, U47 74F257, U48 74HCT4053, U49 MAX232, U5 74F32, U50 NJM4580, U6 74F21, U7 74ALS139, U8 74ALS139, U9 74F138, Y1 30.875

Commit message: initial PCB component layout
Parts:
- added C30: 100n, Capacitor_THT:C_Rect_L7.0mm_W2.5mm_P5.00mm, F.Cu at (96.5, 438.1)
- added C31: 100n, Capacitor_THT:C_Rect_L7.0mm_W2.5mm_P5.00mm, F.Cu at (100.3, 442.0)
- added D4: 1N6263, Diode_THT:D_DO-35_SOD27_P7.62mm_Horizontal, F.Cu at (147.3, 184.2)
- added D5: 1N6263, Diode_THT:D_DO-35_SOD27_P7.62mm_Horizontal, F.Cu at (149.9, 184.2)
- added F1: 2A, Fuse:Fuse_BelFuse_0ZRE0012FF_L8.3mm_W3.8mm, F.Cu at (148.6, 237.5)
- added MH1: MountingHole_2.5mm, MountingHole:MountingHole_2.5mm, F.Cu at (59.7, 210.3)
- added MH2: MountingHole_2.5mm, MountingHole:MountingHole_2.5mm, F.Cu at (59.7, 139.7)
- added MH3: MountingHole_2.5mm, MountingHole:MountingHole_2.5mm, F.Cu at (59.7, 69.1)
- added MH4: MountingHole_2.5mm, MountingHole:MountingHole_2.5mm, F.Cu at (143.5, 210.3)
- added MH5: MountingHole_2.5mm, MountingHole:MountingHole_2.5mm, F.Cu at (143.5, 139.7)
- added MH6: MountingHole_2.5mm, MountingHole:MountingHole_2.5mm, F.Cu at (143.5, 69.1)
- added Q3: BS170, Package_TO_SOT_THT:TO-92_HandSolder, F.Cu at (129.5, 68.6)
- added R8: 220k, Resistor_THT:R_Axial_DIN0204_L3.6mm_D1.6mm_P7.62mm_Horizontal, F.Cu at (151.1, 55.9)
- D1: value D_Schottky_ALT -> 1N5339; footprint Diode_THT:D_DO-35_SOD27_P7.62mm_Horizontal -> Diode_THT:D_5W_P10.16mm_Horizontal
- D2, D3: value D_Schottky_ALT -> 1N6263
- Q1: value DS1233-15 -> DS1233
- Q2: value BS170 -> 2N3904
- R6: value 560k -> 1k
- R7: value 220k -> 560k
- RN8: value 4610X-R2R-103LF -> R2R10k
- SW1: footprint Button_Switch_THT:SW_PUSH-12mm_Wuerth-430476085716 -> FSMRA3JH04:SWITCH_FSMRA3JH04
- U12: value 16R4 -> PAL16R4
- U47: value 74F257 -> 74F157
- Y1: value 30.875 -> 30M875
- moved U50 287.9 mm to (161.3, 53.3), turned to 180 degrees
- moved R7 284.4 mm to (153.7, 63.5), turned to 90 degrees
- moved R5 278.2 mm to (158.8, 55.9), turned to 270 degrees
- moved U33 274.0 mm to (40.6, 45.7)
- moved C2 272.7 mm to (138.4, 47.0), turned to 90 degrees
- moved RN1 272.2 mm to (74.9, 77.5), turned to 270 degrees
- moved R2 271.9 mm to (135.9, 40.6), turned to 270 degrees
- moved U31 265.9 mm to (124.5, 48.3)
- moved J3 263.6 mm to (158.8, 45.7), turned to 270 degrees
- moved R1 263.3 mm to (135.9, 63.5), turned to 270 degrees
- moved Y1 263.2 mm to (137.2, 58.4), turned to 90 degrees
- moved C1 253.1 mm to (138.4, 64.8), turned to 270 degrees
- moved C7 244.5 mm to (143.5, 57.1), turned to 270 degrees
- moved U42 242.8 mm to (63.5, 43.2)
- moved U41 242.6 mm to (52.1, 43.2)
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Connections:
- net Net-(U32-Pad6) renamed /GPU/~cle
- D1 pad 1: mode0 -> 1
- D1 pad 2: Net-(D1-Pad2) -> 0
- D2 pad 1: mode1 -> mode0
- D2 pad 2: Net-(D1-Pad2) -> Net-(D2-Pad2)
- D3 pad 1: Ei2 -> mode1
- D3 pad 2: vblank -> Net-(D2-Pad2)
- J1 pad 1: 1 -> Net-(F1-Pad1)
- J1 pad 3: 1 -> Net-(F1-Pad1)
- J7 pad 10: DD4 -> DD7
- J7 pad 11: DD5 -> DD6
- J7 pad 12: DD6 -> DD5
- J7 pad 13: DD7 -> DD4
- Q2 pad 1: Net-(C4-Pad1) -> 0
- Q2 pad 2: hblank -> Net-(D4-Pad1)
- Q2 pad 3: adac -> Ei2
- R1 pad 2: cclk -> Net-(R1-Pad2)
- R2 pad 1: cclk -> Net-(R1-Pad2)
- R3 pad 2: Net-(D1-Pad2) -> Net-(D2-Pad2)
- R4 pad 1: Net-(C4-Pad1) -> 1
- R4 pad 2: Net-(C5-Pad1) -> Ei2
- R5 pad 1: Net-(C5-Pad1) -> Net-(C4-Pad1)
- R5 pad 2: Net-(C6-Pad1) -> Net-(C5-Pad1)
- R6 pad 1: Net-(C7-Pad2) -> Net-(C5-Pad1)
- R6 pad 2: Net-(R6-Pad2) -> Net-(C6-Pad1)
- R7 pad 1: Net-(R6-Pad2) -> Net-(C7-Pad2)
- R7 pad 2: GNDA -> Net-(R7-Pad2)
- RN7 pad 1: Net-(RN7-Pad1) -> vdac1r
- RN7 pad 2: vdac1r -> Net-(RN7-Pad2)
- RN7 pad 3: Net-(RN7-Pad3) -> vdac1g
- RN7 pad 4: vdac1g -> Net-(RN7-Pad4)
- RN7 pad 5: Net-(RN7-Pad5) -> vdac1b
- RN7 pad 6: vdac1b -> Net-(RN7-Pad6)
- U31 pad 1: Net-(C1-Pad1) -> Net-(U31-Pad1)
- U31 pad 2: cclk -> Net-(U31-Pad2)
- U31 pad 3: cclk -> Net-(C1-Pad1)
- U31 pad 4: dclk -> Net-(R1-Pad2)
- U31 pad 5: Net-(U31-Pad5) -> Net-(R1-Pad2)
- U31 pad 6: Net-(U31-Pad6) -> cclk
- U31 pad 8: Net-(U31-Pad8) -> dclk
- U31 pad 9: Net-(U31-Pad10) -> cclk
- U32 pad 2: Net-(U31-Pad6) -> Net-(U31-Pad2)
- U33 pad 12: tclk -> mode1
- U33 pad 13: mode1 -> tclk
- U34 pad 11: Net-(U33-Pad11) -> nclk
- U34 pad 9: nclk -> Net-(U33-Pad11)
- U35 pad 9: Net-(U31-Pad6) -> Net-(U31-Pad2)
- U36 pad 15: Net-(U31-Pad5) -> Net-(U31-Pad1)
- U41 pad 10: Net-(U31-Pad5) -> Net-(U31-Pad1)
- U42 pad 1: Net-(U31-Pad6) -> Net-(U31-Pad2)
- U47 pad 10: 1 -> C6
- U47 pad 11: 1 -> C2
- U47 pad 12: Net-(RN7-Pad5) -> Net-(U47-Pad12)
- U47 pad 13: C6 -> 1
- U47 pad 14: C2 -> 1
- U47 pad 15: vblank -> 0
- U47 pad 4: Net-(RN7-Pad1) -> Net-(RN7-Pad2)
- U47 pad 7: Net-(RN7-Pad3) -> Net-(RN7-Pad4)
- U47 pad 9: Net-(U47-Pad9) -> Net-(RN7-Pad6)
- U48 pad 10: Net-(D1-Pad2) -> Net-(D2-Pad2)
- U48 pad 11: Net-(D1-Pad2) -> Net-(D2-Pad2)
- U48 pad 9: Net-(D1-Pad2) -> Net-(D2-Pad2)
- U50 pad 1: Net-(C5-Pad2) -> Net-(J3-PadS)
- U50 pad 2: Net-(C5-Pad2) -> Net-(J3-PadS)
- U50 pad 3: Net-(C6-Pad1) -> Net-(R7-Pad2)
- U50 pad 5: Net-(R6-Pad2) -> Net-(C6-Pad1)
- U50 pad 6: Net-(J3-PadS) -> Net-(C5-Pad2)
- U50 pad 7: Net-(J3-PadS) -> Net-(C5-Pad2)
Other:
- board size 203.2 x 127 mm -> 127 x 203.2 mm
- net class Default: clearance 0.2 -> 0.1778; trace_width 0.25 -> 0.2032; via_dia 0.8 -> 0.6; via_drill 0.4 -> 0.3
- rule trace_clearance: 0.2 -> 0.1778
- rule trace_min: 0.2 -> 0.2032
- rule via_min_size: 0.4 -> 0.6

Commit message: v1 schematic/pcb layout after redesign
Parts:
- removed D2, D3, D4, D5: 1N6263, Diode_THT:D_DO-35_SOD27_P7.62mm_Horizontal
- removed R3, R4: 1k, Resistor_THT:R_Axial_DIN0204_L3.6mm_D1.6mm_P7.62mm_Horizontal
- removed U44, U46: 74F574, Package_DIP:DIP-20_W7.62mm_LongPads
- removed U45: 74F299, Package_DIP:DIP-20_W7.62mm_LongPads
- removed U47: 74F157, Package_DIP:DIP-16_W7.62mm_LongPads
- removed U48: 74HCT4053, Package_DIP:DIP-16_W7.62mm_LongPads
- removed U49: MAX232, Package_DIP:DIP-16_W7.62mm_LongPads
- removed U50: NJM4580, Package_SIP:SIP-8_19x3mm_P2.54mm
- added Q4: BS170, Package_TO_SOT_THT:TO-92_HandSolder, F.Cu at (141.0, 45.7)
- added R10: 220k, Resistor_THT:R_Axial_DIN0204_L3.6mm_D1.6mm_P7.62mm_Horizontal, F.Cu at (153.7, 55.9)
- added R9: 560k, Resistor_THT:R_Axial_DIN0204_L3.6mm_D1.6mm_P7.62mm_Horizontal, F.Cu at (156.2, 63.5)
- added RN10: 820, Resistor_THT:R_Array_SIP6, F.Cu at (147.3, 78.7)
- added RN11: R2R10k, Resistor_THT:R_Array_SIP10, F.Cu at (100.3, 43.2)
- added RN9: 1800, Resistor_THT:R_Array_SIP8, F.Cu at (139.7, 76.2)
- Q3: value BS170 -> 2N3904
- R7: value 560k -> 1k
- R8: value 220k -> 1k
- RN4, RN5: value 1800 -> 270; footprint Resistor_THT:R_Array_SIP8 -> Resistor_THT:R_Array_SIP9
- RN6: value 820 -> 270; footprint Resistor_THT:R_Array_SIP6 -> Resistor_THT:R_Array_SIP9
- RN8: value R2R10k -> 1800; footprint Resistor_THT:R_Array_SIP10 -> Resistor_THT:R_Array_SIP8
- U1: value 27C020 -> 74F00; footprint Package_DIP:DIP-32_W15.24mm_LongPads -> Package_DIP:DIP-14_W7.62mm_LongPads
- U10: value 74F138 -> 74LS174
- U11: value 74F157 -> 74F574; footprint Package_DIP:DIP-16_W7.62mm_LongPads -> Package_DIP:DIP-20_W7.62mm_LongPads
- U12: value PAL16R4 -> 74F574
- U13: value 74F574 -> 74F138; footprint Package_DIP:DIP-20_W7.62mm_LongPads -> Package_DIP:DIP-16_W7.62mm_LongPads
- U14: value 74F574 -> PAL16R4
- U15: value 74F163 -> 27C020; footprint Package_DIP:DIP-16_W7.62mm_LongPads -> Package_DIP:DIP-32_W15.24mm_LongPads
- U16: value 74F163 -> AS6C4008; footprint Package_DIP:DIP-16_W7.62mm_LongPads -> Package_DIP:DIP-32_W15.24mm_LongPads
- U17, U22, U37: value 74F541 -> 74F574
- U19: value 74F257 -> 74F163
- U2: value 74F00 -> 74F08
- U20: value 74F574 -> 74F163; footprint Package_DIP:DIP-20_W7.62mm_LongPads -> Package_DIP:DIP-16_W7.62mm_LongPads
- U21: value 74F574 -> 74F541
- U23: value 74F244 -> 74F574
- U24: value 74F574 -> 74F257; footprint Package_DIP:DIP-20_W7.62mm_LongPads -> Package_DIP:DIP-16_W7.62mm_LongPads
- U28: value AS6C4008 -> 74F574; footprint Package_DIP:DIP-32_W15.24mm_LongPads -> Package_DIP:DIP-20_W7.62mm_LongPads
- U29: value 74F574 -> 74F244
- U30: value 74F175 -> 74F541; footprint Package_DIP:DIP-16_W7.62mm_LongPads -> Package_DIP:DIP-20_W7.62mm_LongPads
- U31: value 74F04 -> 74F163; footprint Package_DIP:DIP-14_W7.62mm_LongPads -> Package_DIP:DIP-16_W7.62mm_LongPads
- U32: value 74F00 -> 74F163; footprint Package_DIP:DIP-14_W7.62mm_LongPads -> Package_DIP:DIP-16_W7.62mm_LongPads
- U33: value 74F32 -> 74F541; footprint Package_DIP:DIP-14_W7.62mm_LongPads -> Package_DIP:DIP-20_W7.62mm_LongPads
- U34: value 74F11 -> 74F574; footprint Package_DIP:DIP-14_W7.62mm_LongPads -> Package_DIP:DIP-20_W7.62mm_LongPads
- U35: value 74F163 -> 74F574; footprint Package_DIP:DIP-16_W7.62mm_LongPads -> Package_DIP:DIP-20_W7.62mm_LongPads
- U36: value 74LS163 -> 74F541; footprint Package_DIP:DIP-16_W7.62mm_LongPads -> Package_DIP:DIP-20_W7.62mm_LongPads
- U38: value 74F163 -> 74F299; footprint Package_DIP:DIP-16_W7.62mm_LongPads -> Package_DIP:DIP-20_W7.62mm_LongPads
- U39: value 74LS163 -> 74F574; footprint Package_DIP:DIP-16_W7.62mm_LongPads -> Package_DIP:DIP-20_W7.62mm_LongPads
- U40: value 74F541 -> 74F157; footprint Package_DIP:DIP-20_W7.62mm_LongPads -> Package_DIP:DIP-16_W7.62mm_LongPads
- U41: value 74F163 -> 74HCT4053
- U42: value 74F153 -> MAX232
- U43: value 74F541 -> NJM4580; footprint Package_DIP:DIP-20_W7.62mm_LongPads -> Package_SIP:SIP-8_19x3mm_P2.54mm
- U6: value 74F21 -> 74F32
- U9: value 74F138 -> 74F175
- Y1: value 30M875 -> 32M
- moved C31 224.6 mm to (121.9, 218.4), turned to 270 degrees
- moved C29 223.8 mm to (55.9, 221.0), turned to 270 degrees
- moved C30 219.8 mm to (88.9, 218.4), turned to 270 degrees
- moved U3 177.1 mm to (73.7, 45.7)
- moved R5 148.0 mm to (144.8, 203.2), turned to 90 degrees
- moved RN5 144.1 mm to (63.5, 177.8)
- moved R6 140.4 mm to (142.2, 203.2)
- moved U6 140.0 mm to (58.4, 45.7)
- moved RN6 133.7 mm to (94.0, 186.7)
- moved Q3 129.9 mm to (149.9, 196.8), turned to 90 degrees
- moved U42 124.8 mm to (152.4, 130.8)
- moved SW1 122.1 mm to (40.6, 210.8), turned to 270 degrees
- moved C3 109.4 mm to (47.0, 213.4)
- moved U30 108.6 mm to (43.2, 109.2)
- moved U41 105.7 mm to (141.0, 100.3)
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Connections:
- J7 pad 16: 1 -> qclk1
- J7 pad 17: 1 -> eclk
- J7 pad 18: pclk1 -> ~eoe
- J7 pad 19: qclk1 -> I0
- J7 pad 2: PD0 -> PD7
- J7 pad 20: eclk -> I1
- J7 pad 21: ~eoe -> I2
- J7 pad 3: PD1 -> PD6
- J7 pad 4: PD2 -> PD5
- J7 pad 5: PD3 -> PD4
- J7 pad 6: PD4 -> PD3
- J7 pad 7: PD5 -> PD2
- J7 pad 8: PD6 -> PD1
- J7 pad 9: PD7 -> PD0
- Q2 pad 2: Net-(D4-Pad1) -> Eo2
- Q3 pad 1: Net-(C4-Pad1) -> 0
- Q3 pad 2: hblank -> Eo3
- Q3 pad 3: adac -> Ei3
- R1 pad 2: Net-(R1-Pad2) -> cclk
- R2 pad 1: Net-(R1-Pad2) -> cclk
- R5 pad 1: Net-(C4-Pad1) -> 1
- R5 pad 2: Net-(C5-Pad1) -> Ei3
- R6 pad 1: Net-(C5-Pad1) -> 1
- R6 pad 2: Net-(C6-Pad1) -> Ei2
- R7 pad 1: Net-(C7-Pad2) -> Net-(C4-Pad1)
- R7 pad 2: Net-(R7-Pad2) -> Net-(C5-Pad1)
- R8 pad 1: Net-(R7-Pad2) -> Net-(C5-Pad1)
- R8 pad 2: GNDA -> Net-(C6-Pad1)
- RN4 pad 1: vdac0r -> 0
- RN4 pad 2: C0 -> PA0
- RN4 pad 3: C1 -> PA1
- RN4 pad 4: C1 -> PA2
- RN4 pad 5: C2 -> PA3
- RN4 pad 6: C2 -> PA4
- RN4 pad 7: C2 -> PA5
- RN4 pad 8: C2 -> PA6
- RN5 pad 1: vdac0g -> 1
- RN5 pad 2: C3 -> /CPU/HL0
- RN5 pad 3: C4 -> /CPU/HL1
- RN5 pad 4: C4 -> /CPU/HL2
- RN5 pad 5: C5 -> /CPU/HL3
- RN5 pad 6: C5 -> /CPU/HL4
- RN5 pad 7: C5 -> /CPU/HL5
- RN5 pad 8: C5 -> /CPU/HL6
- RN6 pad 1: vdac0b -> 1
- RN6 pad 2: C6 -> I8
- RN6 pad 3: C6 -> I9
- RN6 pad 4: vdac0b -> I10
- RN6 pad 5: vdac0b -> I11
- RN6 pad 6: C7 -> I12
- RN8 pad 1: adac -> vdac2r
- RN8 pad 2: /GPU/G7 -> C0
- RN8 pad 3: /GPU/G6 -> C1
- RN8 pad 4: /GPU/G5 -> C1
- RN8 pad 5: /GPU/G4 -> C2
- RN8 pad 6: /GPU/G3 -> C2
- RN8 pad 7: /GPU/G2 -> C2
- RN8 pad 8: /GPU/G1 -> C2
- U1 pad 1: 1 -> Net-(C1-Pad1)
- U1 pad 10: PA2 -> Net-(U1-Pad10)
- U1 pad 11: PA1 -> hblank
- U1 pad 12: PA0 -> Net-(U1-Pad12)
- U1 pad 13: PD0 -> Net-(U1-Pad12)
- U1 pad 14: PD1 -> 1
- U1 pad 2: PA16 -> Net-(C1-Pad1)
- U1 pad 3: PA15 -> cclk
- U1 pad 4: PA12 -> cclk
- U1 pad 5: PA7 -> cclk
- U1 pad 6: PA6 -> dclk
- U1 pad 7: PA5 -> 0
- U1 pad 8: PA4 -> /GPU/~cle
- U1 pad 9: PA3 -> cclk
- U10 pad 1: I3 -> 1
- U10 pad 10: ~xroe -> ~pgoe
- U10 pad 12: Net-(U10-Pad12) -> ~pcoe
- U10 pad 15: Net-(U10-Pad15) -> ~alue
- U10 pad 2: I4 -> Net-(U10-Pad2)
- U10 pad 3: Net-(U10-Pad3) -> ~inst
- U10 pad 4: pclk1 -> Net-(U10-Pad4)
- U10 pad 5: ~1st -> ~voe
- U10 pad 6: 1 -> Net-(U10-Pad6)
- U10 pad 7: ~eoe -> ~xoe
- U10 pad 9: Net-(U10-Pad9) -> dclk
- U11 pad 1: pclk1 -> 0
- U11 pad 10: Net-(U11-Pad10) -> 0
- U11 pad 11: hblank -> ~ille
- U11 pad 12: DA16 -> I7
- U11 pad 13: 1 -> I6
- U11 pad 14: I4 -> I5
- U11 pad 15: 0 -> I4
- U11 pad 16: 1 -> I3
- U11 pad 2: 0 -> PD0
- U11 pad 3: ~inst -> PD1
- U11 pad 4: Net-(U11-Pad4) -> PD2
- U11 pad 5: 1 -> PD3
- U11 pad 6: ~inst -> PD4
- U11 pad 7: ~ile -> PD5
- U11 pad 8: 0 -> PD6
- U11 pad 9: PA16 -> PD7
- U12 pad 1: sclk -> I7
- U12 pad 11: 0 -> ~ihle
- U12 pad 12: ~rst -> I15
- U12 pad 13: pcent -> I14
- U12 pad 14: ~inst -> I13
- U12 pad 15: hsel -> I12
- U12 pad 16: boot -> I11
- U12 pad 17: Net-(U12-Pad17) -> I10
- U12 pad 18: Net-(U11-Pad10) -> I9
- U12 pad 19: pclk1 -> I8
- U12 pad 2: I0 -> PD0
- U12 pad 3: I1 -> PD1
- U12 pad 4: I2 -> PD2
- U12 pad 5: I3+4 -> PD3
- U12 pad 6: I5 -> PD4
- U12 pad 7: I6 -> PD5
- U12 pad 8: I7 -> PD6
- U12 pad 9: DD7 -> PD7
- U13 pad 1: 0 -> I0
- U13 pad 10: 0 -> ~ele
- U13 pad 11: ~ile -> ~hlle
- U13 pad 12: I7 -> ~vle
- U13 pad 13: I6 -> ~scle
- U13 pad 14: I5 -> ~pcle
- U13 pad 15: I4 -> ~pgle
- U13 pad 16: I3 -> 1
- U13 pad 2: PD0 -> I1
- U13 pad 3: PD1 -> I2
- U13 pad 4: PD2 -> qclk1
- U13 pad 5: PD3 -> ~rom2
- U13 pad 6: PD4 -> I15
- U13 pad 7: PD5 -> ~yle
- U13 pad 8: PD6 -> 0
- U13 pad 9: PD7 -> ~xle
- U14 pad 1: 0 -> Net-(U14-Pad1)
- U14 pad 11: dclk -> 0
- U14 pad 12: ~xoe -> DD7
- U14 pad 13: Net-(U14-Pad13) -> ~hloe
- U14 pad 14: ~gcoe -> ~inst
- U14 pad 15: ~fnoe -> hsel
- U14 pad 16: ~alue -> boot
- U14 pad 17: ~pcoe -> Net-(U14-Pad17)
- U14 pad 18: ~pgoe -> pcent
- U14 pad 19: ~1st -> PA16
- U14 pad 2: ~inst -> ~rst
- U14 pad 3: Net-(U14-Pad3) -> pclk1
- U14 pad 4: Net-(U14-Pad4) -> hblank
- U14 pad 5: Net-(U14-Pad5) -> I3
- U14 pad 6: Net-(U14-Pad6) -> I4
- U14 pad 7: sclk -> I5
- U14 pad 8: Net-(U14-Pad8) -> I6
- U14 pad 9: Net-(U14-Pad13) -> I7
- U15 pad 1: ~pcmr -> 1
- U15 pad 10: pcent -> PA2
- U15 pad 11: /CPU/PC3 -> PA1
- U15 pad 12: /CPU/PC2 -> PA0
- U15 pad 13: /CPU/PC1 -> PD0
- U15 pad 14: /CPU/PC0 -> PD1
- U15 pad 15: Net-(U15-Pad15) -> PD2
- U15 pad 16: 1 -> 0
- U15 pad 2: mclk -> PA16
- U15 pad 3: PD0 -> PA15
- U15 pad 4: PD1 -> PA12
- U15 pad 5: PD2 -> PA7
- U15 pad 6: PD3 -> PA6
- U15 pad 7: 1 -> PA5
- U15 pad 8: 0 -> PA4
- U15 pad 9: ~pcpe -> PA3
- U16 pad 1: ~pcmr -> DA18
- U16 pad 10: Net-(U15-Pad15) -> DA2
- U16 pad 11: /CPU/PC7 -> DA1
- U16 pad 12: /CPU/PC6 -> DA0
- U16 pad 13: /CPU/PC5 -> DD0
- U16 pad 14: /CPU/PC4 -> DD1
- U16 pad 15: Net-(U16-Pad15) -> DD2
- U16 pad 16: 1 -> 0
- U16 pad 2: mclk -> DA16
- U16 pad 3: PD4 -> DA14
- U16 pad 4: PD5 -> DA12
- U16 pad 5: PD6 -> DA7
- U16 pad 6: PD7 -> DA6
- U16 pad 7: 1 -> DA5
- U16 pad 8: 0 -> DA4
- U16 pad 9: ~pcpe -> DA3
- U17 pad 1: ~pcoe -> pclk1
- U17 pad 11: PA7 -> qclk1
- U17 pad 12: PA6 -> PA7
- U17 pad 13: PA5 -> PA6
- U17 pad 14: PA4 -> PA5
- U17 pad 15: PA3 -> PA4
- U17 pad 16: PA2 -> PA3
- U17 pad 17: PA1 -> PA2
- U17 pad 18: PA0 -> PA1
- U17 pad 19: ~pcoe -> PA0
- U17 pad 2: /CPU/PC0 -> DD0
- U17 pad 3: /CPU/PC1 -> DD1
- U17 pad 4: /CPU/PC2 -> DD2
- U17 pad 5: /CPU/PC3 -> DD3
- U17 pad 6: /CPU/PC4 -> DD4
- U17 pad 7: /CPU/PC5 -> DD5
- U17 pad 8: /CPU/PC6 -> DD6
- U17 pad 9: /CPU/PC7 -> DD7
- U18 pad 1: ~pgoe -> ~alue
- U18 pad 11: ~pgle -> pclk1
- U18 pad 12: PA15 -> PA7
- U18 pad 13: PA14 -> PA6
- U18 pad 14: PA13 -> PA5
- U18 pad 15: PA12 -> PA4
- U18 pad 16: PA11 -> PA3
- U18 pad 17: PA10 -> PA2
- U18 pad 18: PA9 -> PA1
- U18 pad 19: PA8 -> PA0
- U18 pad 2: PD0 -> DD0
- U18 pad 3: PD1 -> DD1
- U18 pad 4: PD2 -> DD2
- U18 pad 5: PD3 -> DD3
- U18 pad 6: PD4 -> DD4
- U18 pad 7: PD5 -> DD5
- U18 pad 8: PD6 -> DD6
- U18 pad 9: PD7 -> DD7
- U19 pad 1: hsel -> ~pcmr
- U19 pad 10: /CPU/HL7 -> pcent
- U19 pad 11: /CPU/HL3 -> /CPU/PC3
- U19 pad 12: PA10 -> /CPU/PC2
- U19 pad 13: /CPU/HL6 -> /CPU/PC1
- U19 pad 14: /CPU/HL2 -> /CPU/PC0
- U19 pad 15: ~alue -> Net-(U19-Pad15)
- U19 pad 2: /CPU/HL0 -> mclk
- U19 pad 3: /CPU/HL4 -> PD0
- U19 pad 4: PA8 -> PD1
- U19 pad 5: /CPU/HL1 -> PD2
- U19 pad 6: /CPU/HL5 -> PD3
- U19 pad 7: PA9 -> 1
- U19 pad 9: PA11 -> ~pcle
- U2 pad 1: rclk -> sclk
- U2 pad 10: ~bra -> I6
- U2 pad 11: DA18 -> ~aoe
- U2 pad 12: qclk1 -> ~ram2
- U2 pad 13: /CPU/Eo3 -> Net-(U2-Pad13)
- U2 pad 2: Net-(U2-Pad2) -> ~rst
- U2 pad 3: Net-(U14-Pad4) -> Net-(U14-Pad1)
- U2 pad 4: Net-(U2-Pad4) -> ~pgle
- U2 pad 5: Net-(U2-Pad5) -> ~rst
- U2 pad 6: Net-(U2-Pad6) -> ~pcmr
- U2 pad 9: ~1st -> ~inst
- U20 pad 1: 0 -> ~pcmr
- U20 pad 10: 0 -> Net-(U19-Pad15)
- U20 pad 11: ~hlle -> /CPU/PC7
- U20 pad 12: /CPU/HL7 -> /CPU/PC6
- U20 pad 13: /CPU/HL6 -> /CPU/PC5
- U20 pad 14: /CPU/HL5 -> /CPU/PC4
- U20 pad 15: /CPU/HL4 -> Net-(U20-Pad15)
- U20 pad 16: /CPU/HL3 -> 1
- U20 pad 2: PD0 -> mclk
- U20 pad 3: PD1 -> PD4
- U20 pad 4: PD2 -> PD5
- U20 pad 5: PD3 -> PD6
- U20 pad 6: PD4 -> PD7
- U20 pad 7: PD5 -> 1
- U20 pad 8: PD6 -> 0
- U20 pad 9: PD7 -> ~pcle
- U21 pad 1: ~aoe -> ~pcoe
- U21 pad 11: ~alue -> PA7
- U21 pad 12: DD7 -> PA6
- U21 pad 13: DD6 -> PA5
- U21 pad 14: DD5 -> PA4
- U21 pad 15: DD4 -> PA3
- U21 pad 16: DD3 -> PA2
- U21 pad 17: DD2 -> PA1
- U21 pad 18: DD1 -> PA0
- U21 pad 19: DD0 -> ~pcoe
- U21 pad 2: PD0 -> /CPU/PC0
- U21 pad 3: PD1 -> /CPU/PC1
- U21 pad 4: PD2 -> /CPU/PC2
- U21 pad 5: PD3 -> /CPU/PC3
- U21 pad 6: PD4 -> /CPU/PC4
- U21 pad 7: PD5 -> /CPU/PC5
- U21 pad 8: PD6 -> /CPU/PC6
- U21 pad 9: PD7 -> /CPU/PC7
- U22 pad 1: ~xroe -> ~pgoe
- U22 pad 11: DD7 -> ~pgle
- U22 pad 12: DD6 -> PA15
- U22 pad 13: DD5 -> PA14
- U22 pad 14: DD4 -> PA13
- U22 pad 15: DD3 -> PA12
- U22 pad 16: DD2 -> PA11
- U22 pad 17: DD1 -> PA10
- U22 pad 18: DD0 -> PA9
- U22 pad 19: ~xroe -> PA8
- U22 pad 2: DA0 -> PD0
- U22 pad 3: DA1 -> PD1
- U22 pad 4: DA2 -> PD2
- U22 pad 5: DA3 -> PD3
- U22 pad 6: DA4 -> PD4
- U22 pad 7: DA5 -> PD5
- U22 pad 8: DA6 -> PD6
- U22 pad 9: DA7 -> PD7
- U23 pad 1: ~eoe -> ~hloe
- U23 pad 11: I0 -> ~hlle
- U23 pad 12: DD3 -> /CPU/HL7
- U23 pad 13: I1 -> /CPU/HL6
- U23 pad 14: DD2 -> /CPU/HL5
- U23 pad 15: I2 -> /CPU/HL4
- U23 pad 16: DD1 -> /CPU/HL3
- U23 pad 17: I6 -> /CPU/HL2
- U23 pad 18: DD0 -> /CPU/HL1
- U23 pad 19: ~fnoe -> /CPU/HL0
- U23 pad 2: Ei0 -> PD0
- U23 pad 3: PA15 -> PD1
- U23 pad 4: Ei1 -> PD2
- U23 pad 5: PA14 -> PD3
- U23 pad 6: Ei2 -> PD4
- U23 pad 7: PA13 -> PD5
- U23 pad 8: Ei3 -> PD6
- U23 pad 9: PA12 -> PD7
- U24 pad 1: ~alue -> hsel
- U24 pad 10: 0 -> /CPU/HL7
- U24 pad 11: pclk1 -> /CPU/HL3
- U24 pad 12: PA7 -> PA10
- U24 pad 13: PA6 -> /CPU/HL6
- U24 pad 14: PA5 -> /CPU/HL2
- U24 pad 15: PA4 -> ~alue
- U24 pad 16: PA3 -> 1
- U24 pad 2: DD0 -> /CPU/HL0
- U24 pad 3: DD1 -> /CPU/HL4
- U24 pad 4: DD2 -> PA8
- U24 pad 5: DD3 -> /CPU/HL1
- U24 pad 6: DD4 -> /CPU/HL5
- U24 pad 7: DD5 -> PA9
- U24 pad 8: DD6 -> 0
- U24 pad 9: DD7 -> PA11
- U25 pad 1: ~gcoe -> 0
- U25 pad 11: qclk1 -> ~ele
- U25 pad 12: PA7 -> Net-(U25-Pad12)
- U25 pad 13: PA6 -> Eo6
- U25 pad 14: PA5 -> Eo5
- U25 pad 15: PA4 -> Eo4
- U25 pad 16: PA3 -> Eo3
- U25 pad 17: PA2 -> Eo2
- U25 pad 18: PA1 -> Eo1
- U25 pad 19: PA0 -> Eo0
- U25 pad 2: DD0 -> PD0
- U25 pad 3: DD1 -> PD1
- U25 pad 4: DD2 -> PD2
- U25 pad 5: DD3 -> PD3
- U25 pad 6: DD4 -> PD4
- U25 pad 7: DD5 -> PD5
- U25 pad 8: DD6 -> PD6
- U25 pad 9: DD7 -> PD7
- U28 pad 1: DA18 -> ~aoe
- U28 pad 10: DA2 -> 0
- U28 pad 11: DA1 -> ~alue
- U28 pad 12: DA0 -> DD7
- U28 pad 13: DD0 -> DD6
- U28 pad 14: DD1 -> DD5
- U28 pad 15: DD2 -> DD4
- U28 pad 16: 0 -> DD3
- U28 pad 17: DD3 -> DD2
- U28 pad 18: DD4 -> DD1
- U28 pad 19: DD5 -> DD0
- U28 pad 2: DA16 -> PD0
- U28 pad 20: DD6 -> 1
- U28 pad 3: DA14 -> PD1
- U28 pad 4: DA12 -> PD2
- U28 pad 5: DA7 -> PD3
- U28 pad 6: DA6 -> PD4
- U28 pad 7: DA5 -> PD5
- U28 pad 8: DA4 -> PD6
- U28 pad 9: DA3 -> PD7
- U29 pad 1: 0 -> ~eoe
- U29 pad 11: ~ele -> I8
- U29 pad 12: mode1 -> DD3
- U29 pad 13: mode0 -> I9
- U29 pad 14: vblank -> DD2
- U29 pad 15: vsync -> I10
- U29 pad 16: /CPU/Eo3 -> DD1
- U29 pad 17: /CPU/Eo2 -> I11
- U29 pad 18: Eo1 -> DD0
- U29 pad 19: Eo0 -> ~alue
- U29 pad 2: PD0 -> Ei0
- U29 pad 3: PD1 -> PA15
- U29 pad 4: PD2 -> Ei1
- U29 pad 5: PD3 -> PA14
- U29 pad 6: PD4 -> Ei2
- U29 pad 7: PD5 -> PA13
- U29 pad 8: PD6 -> Ei3
- U29 pad 9: PD7 -> PA12
- U3 pad 1: Net-(U3-Pad1) -> qclk2
- U3 pad 10: Net-(U3-Pad10) -> mode1
- U3 pad 11: ~pcmr -> ~doe
- U3 pad 13: ~rst -> qclk1
- U3 pad 2: ~inst -> Net-(U3-Pad2)
- U3 pad 3: Net-(U2-Pad2) -> Net-(U3-Pad3)
- U3 pad 4: Net-(U3-Pad4) -> Net-(U3-Pad3)
- U3 pad 5: I5 -> nclk
- U3 pad 6: Net-(U10-Pad3) -> Net-(U1-Pad10)
- U3 pad 8: ~pcpe -> Net-(U3-Pad8)
- U3 pad 9: ~pcle -> mode0
- U30 pad 1: ~rst -> ~xroe
- U30 pad 10: pclk2 -> 0
- U30 pad 11: qclk2 -> DD7
- U30 pad 12: sclk -> DD6
- U30 pad 13: pclk2 -> DD5
- U30 pad 14: sclk -> DD4
- U30 pad 15: rclk -> DD3
- U30 pad 16: 1 -> DD2
- U30 pad 2: mclk -> DA0
- U30 pad 3: nclk -> DA1
- U30 pad 4: nclk -> DA2
- U30 pad 5: sclk -> DA3
- U30 pad 6: qclk1 -> DA4
- U30 pad 7: pclk1 -> DA5
- U30 pad 8: 0 -> DA6
- U30 pad 9: dclk -> DA7
- U31 pad 1: Net-(U31-Pad1) -> 1
- U31 pad 10: Net-(U31-Pad10) -> 1
- U31 pad 11: 1 -> /GPU/H3
- U31 pad 12: Net-(U31-Pad12) -> /GPU/H2
- U31 pad 13: Net-(U31-Pad13) -> eclk
- U31 pad 14: 1 -> tclk
- U31 pad 2: Net-(U31-Pad2) -> qclk2
- U31 pad 3: Net-(C1-Pad1) -> 0
- U31 pad 4: Net-(R1-Pad2) -> 0
- U31 pad 5: Net-(R1-Pad2) -> 0
- U31 pad 6: cclk -> 0
- U31 pad 7: 0 -> 1
- U31 pad 8: dclk -> 0
- U31 pad 9: cclk -> ~scle
- U32 pad 1: Net-(U32-Pad1) -> 1
- U32 pad 10: SC1 -> Net-(U31-Pad15)
- U32 pad 11: DA17 -> /GPU/H7
- U32 pad 12: qclk1 -> /GPU/H6
- U32 pad 13: /CPU/Eo2 -> /GPU/H5
- U32 pad 14: 1 -> /GPU/H4
- U32 pad 2: Net-(U31-Pad2) -> qclk2
- U32 pad 3: hblank -> 0
- U32 pad 4: cclk -> 1
- U32 pad 5: Net-(U32-Pad5) -> 0
- U32 pad 6: /GPU/~cle -> 0
- U32 pad 7: 0 -> 1
- U32 pad 8: Net-(U31-Pad13) -> 0
- U32 pad 9: SC0 -> ~scle
- U33 pad 1: /GPU/H7 -> hblank
- U33 pad 10: Net-(U33-Pad10) -> 0
- U33 pad 11: Net-(U33-Pad11) -> DA7
- U33 pad 12: mode1 -> DA6
- U33 pad 13: tclk -> DA5
- U33 pad 14: 1 -> DA4
- U33 pad 2: /GPU/H6 -> tclk
- U33 pad 3: Net-(U33-Pad3) -> eclk
- U33 pad 4: Net-(U33-Pad3) -> /GPU/H2
- U33 pad 5: /GPU/H5 -> /GPU/H3
- U33 pad 6: ~hsync -> /GPU/H4
- U33 pad 7: 0 -> /GPU/H5
- U33 pad 8: Net-(U32-Pad1) -> /GPU/H6
- U33 pad 9: Net-(U33-Pad3) -> /GPU/H7
- U34 pad 1: /GPU/H5 -> ~voe
- U34 pad 10: qclk2 -> 1
- U34 pad 11: nclk -> ~vle
- U34 pad 12: Net-(U33-Pad10) -> DA15
- U34 pad 13: /GPU/H3 -> DA14
- U34 pad 14: 1 -> DA13
- U34 pad 2: /GPU/H4 -> PD0
- U34 pad 3: SC0 -> PD1
- U34 pad 4: SC1 -> PD2
- U34 pad 5: SC2 -> PD3
- U34 pad 6: Net-(U34-Pad6) -> PD4
- U34 pad 7: 0 -> PD5
- U34 pad 8: Net-(U32-Pad5) -> PD6
- U34 pad 9: Net-(U33-Pad11) -> PD7
- U35 pad 1: ~rst -> 1
- U35 pad 10: 1 -> 0
- U35 pad 11: /GPU/H3 -> ~scle
- U35 pad 12: /GPU/H2 -> mode1
- U35 pad 13: eclk -> mode0
- U35 pad 14: tclk -> vsync
- U35 pad 15: Net-(U35-Pad15) -> vblank
- U35 pad 16: 1 -> Net-(U35-Pad16)
- U35 pad 2: qclk2 -> PD0
- U35 pad 3: 0 -> PD1
- U35 pad 4: 0 -> PD2
- U35 pad 5: 1 -> PD3
- U35 pad 6: 1 -> PD4
- U35 pad 7: 1 -> PD5
- U35 pad 8: 0 -> PD6
- U35 pad 9: Net-(U31-Pad2) -> PD7
- U36 pad 1: ~rst -> hblank
- U36 pad 10: Net-(U35-Pad15) -> 0
- U36 pad 11: /GPU/H7 -> PA15
- U36 pad 12: /GPU/H6 -> PA14
- U36 pad 13: /GPU/H5 -> PA13
- U36 pad 14: /GPU/H4 -> PA12
- U36 pad 15: Net-(U31-Pad1) -> PA11
- U36 pad 16: 1 -> PA10
- U36 pad 2: qclk2 -> Net-(U35-Pad19)
- U36 pad 3: 0 -> Net-(U35-Pad18)
- U36 pad 4: 0 -> Net-(U35-Pad17)
- U36 pad 5: 0 -> Net-(U35-Pad16)
- U36 pad 6: 0 -> C3
- U36 pad 7: 1 -> C7
- U36 pad 8: 0 -> mode0
- U37 pad 1: hblank -> 0
- U37 pad 11: DA7 -> pclk2
- U37 pad 12: DA6 -> /GPU/G7
- U37 pad 13: DA5 -> /GPU/G6
- U37 pad 14: DA4 -> /GPU/G5
- U37 pad 15: DA3 -> /GPU/G4
- U37 pad 16: DA2 -> /GPU/G3
- U37 pad 17: DA1 -> /GPU/G2
- U37 pad 18: DA0 -> /GPU/G1
- U37 pad 19: qclk2 -> /GPU/G0
- U37 pad 2: tclk -> PD0
- U37 pad 3: eclk -> PD1
- U37 pad 4: /GPU/H2 -> PD2
- U37 pad 5: /GPU/H3 -> PD3
- U37 pad 6: /GPU/H4 -> PD4
- U37 pad 7: /GPU/H5 -> PD5
- U37 pad 8: /GPU/H6 -> PD6
- U37 pad 9: /GPU/H7 -> PD7
- U38 pad 10: Net-(U38-Pad10) -> 0
- U38 pad 11: /GPU/V3 -> 1
- U38 pad 12: /GPU/V2 -> dclk
- U38 pad 13: /GPU/V1 -> /GPU/G1
- U38 pad 14: /GPU/V0 -> /GPU/G3
- U38 pad 15: Net-(U38-Pad15) -> /GPU/G5
- U38 pad 16: 1 -> /GPU/G7
- U38 pad 2: qclk2 -> 1
- U38 pad 3: PD0 -> 1
- U38 pad 4: PD1 -> /GPU/G6
- U38 pad 5: PD2 -> /GPU/G4
- U38 pad 6: PD3 -> /GPU/G2
- U38 pad 7: 1 -> /GPU/G0
- U38 pad 8: 0 -> Net-(U38-Pad8)
- U38 pad 9: ~vle -> 1
- U39 pad 1: 1 -> vblank
- U39 pad 10: Net-(U38-Pad15) -> 0
- U39 pad 11: /GPU/V7 -> /GPU/~cle
- U39 pad 12: /GPU/V6 -> C7
- U39 pad 13: /GPU/V5 -> C6
- U39 pad 14: /GPU/V4 -> C5
- U39 pad 15: Net-(U39-Pad15) -> C4
- U39 pad 16: 1 -> C3
- U39 pad 2: qclk2 -> PA0
- U39 pad 3: PD4 -> PA1
- U39 pad 4: PD5 -> PA2
- U39 pad 5: PD6 -> PA3
- U39 pad 6: PD7 -> PA4
- U39 pad 7: 1 -> PA5
- U39 pad 8: 0 -> PA6
- U39 pad 9: ~vle -> PA7
- U4 pad 1: Net-(U2-Pad2) -> Eo4
- U4 pad 10: Net-(U14-Pad4) -> Net-(U4-Pad10)
- U4 pad 11: ~pgle -> Net-(U4-Pad10)
- U4 pad 12: Net-(U3-Pad12) -> pclk1
- U4 pad 13: qclk1 -> I14
- U4 pad 2: sclk -> Net-(U4-Pad10)
- U4 pad 3: Net-(U14-Pad5) -> DA16
- U4 pad 4: Net-(U14-Pad5) -> Eo5
- U4 pad 5: Net-(U2-Pad6) -> Net-(U4-Pad10)
- U4 pad 6: Net-(U14-Pad6) -> DA17
- U4 pad 8: Net-(U14-Pad3) -> DA18
- U4 pad 9: boot -> Eo6
- U40 pad 1: hblank -> Net-(U38-Pad17)
- U40 pad 10: 0 -> C6
- U40 pad 11: DA15 -> C2
- U40 pad 12: DA14 -> Net-(U40-Pad12)
- U40 pad 13: DA13 -> 1
- U40 pad 14: DA12 -> 1
- U40 pad 15: DA11 -> vblank
- U40 pad 16: DA10 -> 1
- U40 pad 2: /GPU/V0 -> C0
- U40 pad 3: /GPU/V1 -> C4
- U40 pad 4: /GPU/V2 -> Net-(RN7-Pad2)
- U40 pad 5: /GPU/V3 -> C1
- U40 pad 6: /GPU/V4 -> C5
- U40 pad 7: /GPU/V5 -> Net-(RN7-Pad4)
- U40 pad 8: /GPU/V6 -> 0
- U40 pad 9: /GPU/V7 -> Net-(RN7-Pad6)
- U41 pad 1: ~rst -> vdac2g
- U41 pad 10: Net-(U31-Pad1) -> Net-(U3-Pad8)
- U41 pad 11: Net-(U41-Pad11) -> Net-(U3-Pad8)
- U41 pad 12: SC2 -> vdac1r
- U41 pad 13: SC1 -> vdac2r
- U41 pad 14: SC0 -> Net-(J6-Pad2)
- U41 pad 15: Net-(U41-Pad15) -> Net-(J6-Pad1)
- U41 pad 16: 1 -> VDD
- U41 pad 2: qclk2 -> vdac1g
- U41 pad 3: 0 -> vdac2b
- U41 pad 4: 0 -> Net-(J6-Pad3)
- U41 pad 5: 0 -> vdac1b
- U41 pad 6: 0 -> hblank
- U41 pad 7: 1 -> VEE
- U41 pad 8: 0 -> GNDA
- U41 pad 9: 1 -> Net-(U3-Pad8)
- U42 pad 1: Net-(U31-Pad2) -> Net-(C9-Pad1)
- U42 pad 10: 0 -> Eo1
- U42 pad 11: Net-(U41-Pad11) -> Eo0
- U42 pad 12: 1 -> Ei0
- U42 pad 13: 1 -> Net-(J5-Pad2)
- U42 pad 14: mode0 -> Net-(J5-Pad3)
- U42 pad 2: mode1 -> VDD
- U42 pad 3: Net-(U31-Pad12) -> Net-(C9-Pad2)
- U42 pad 4: SC0 -> Net-(C8-Pad1)
- U42 pad 5: Net-(U41-Pad15) -> Net-(C8-Pad2)
- U42 pad 6: Net-(U34-Pad6) -> VEE
- U42 pad 7: Net-(U38-Pad10) -> Net-(J5-Pad7)
- U42 pad 8: 0 -> Net-(J5-Pad8)
- U42 pad 9: Net-(U42-Pad9) -> Ei1
- U43 pad 1: hblank -> Net-(J3-PadS)
- U43 pad 2: SC0 -> Net-(J3-PadS)
- U43 pad 3: SC1 -> Net-(R10-Pad1)
- U43 pad 4: SC2 -> VEE
- U43 pad 5: Net-(U42-Pad9) -> Net-(C6-Pad1)
- U43 pad 6: C3 -> Net-(C5-Pad2)
- U43 pad 7: C7 -> Net-(C5-Pad2)
- U43 pad 8: mode1 -> VDD
- U5 pad 1: I3 -> hblank
- U5 pad 10: Net-(U5-Pad10) -> Net-(U10-Pad13)
- U5 pad 11: Net-(U5-Pad10) -> ~exle
- U5 pad 12: pclk1 -> ~rom2
- U5 pad 13: Net-(U2-Pad8) -> I15
- U5 pad 2: I4 -> rclk
- U5 pad 3: I3+4 -> Net-(U10-Pad4)
- U5 pad 4: I3+4 -> sclk
- U5 pad 5: Net-(U3-Pad1) -> I13
- U5 pad 6: ~bra -> Net-(U10-Pad6)
- U5 pad 8: ~dwe -> Net-(U10-Pad11)
- U5 pad 9: I3 -> boot
- U6 pad 1: Net-(U5-Pad10) -> I12
- U6 pad 10: Net-(U10-Pad14) -> Net-(U1-Pad12)
- U6 pad 11: (no net) -> Net-(U1-Pad12)
- U6 pad 12: Net-(U10-Pad11) -> /GPU/H6
- U6 pad 13: Net-(U10-Pad9) -> /GPU/H7
- U6 pad 2: Net-(U10-Pad15) -> ~ram2
- U6 pad 3: (no net) -> ~dwe
- U6 pad 4: Net-(U10-Pad13) -> mode1
- U6 pad 5: Net-(U10-Pad12) -> tclk
- U6 pad 6: ~aoe -> Net-(U3-Pad2)
- U6 pad 8: ~doe -> ~hsync
- U6 pad 9: qclk1 -> /GPU/H4
- U7 pad 1: ~bra -> rclk
- U7 pad 10: Net-(U2-Pad4) -> ~eoe
- U7 pad 11: Net-(U3-Pad4) -> ~xroe
- U7 pad 12: Net-(U3-Pad1) -> Net-(U2-Pad13)
- U7 pad 13: I6 -> I4
- U7 pad 14: I5 -> I3
- U7 pad 15: I7 -> ~ram1
- U7 pad 2: I2 -> Net-(U2-Pad8)
- U7 pad 3: Net-(U11-Pad4) -> ~rst
- U7 pad 6: Net-(U3-Pad10) -> Net-(U10-Pad13)
- U7 pad 7: Net-(U3-Pad12) -> Net-(U10-Pad14)
- U7 pad 9: Net-(U2-Pad5) -> Net-(U3-Pad12)
- U8 pad 1: Net-(U3-Pad1) -> qclk1
- U8 pad 10: Net-(U8-Pad10) -> ~rom2
- U8 pad 11: Net-(U8-Pad11) -> ~ram1
- U8 pad 13: Net-(U3-Pad4) -> Net-(U10-Pad2)
- U8 pad 14: ~bra -> qclk1
- U8 pad 15: I7 -> 0
- U8 pad 2: pclk1 -> hsel
- U8 pad 3: I4 -> ~inst
- U8 pad 4: Net-(U8-Pad4) -> ~ille
- U8 pad 5: Net-(U8-Pad5) -> ~ihle
- U8 pad 7: Net-(U14-Pad8) -> Net-(U8-Pad7)
- U8 pad 9: ~r8en -> ~ram2
- U9 pad 1: I0 -> ~rst
- U9 pad 10: ~ele -> pclk2
- U9 pad 11: ~hlle -> qclk2
- U9 pad 12: ~yle -> sclk
- U9 pad 13: ~xle -> pclk2
- U9 pad 14: ~vle -> sclk
- U9 pad 15: ~pcle -> rclk
- U9 pad 2: I1 -> mclk
- U9 pad 3: I2 -> nclk
- U9 pad 4: qclk1 -> nclk
- U9 pad 5: ~r8en -> sclk
- U9 pad 6: ~inst -> qclk1
- U9 pad 7: Net-(U9-Pad7) -> pclk1
- U9 pad 9: ~exle -> dclk
Other:
- net class Default: clearance 0.1778 -> 0.2; trace_width 0.2032 -> 0.25; via_dia 0.6 -> 0.8; via_drill 0.3 -> 0.4
- rule trace_clearance: 0.1778 -> 0.2

Commit message: minor tweaks
Parts:
- removed the RN5 at (63.5, 177.8)
- RN10: value 820 -> 1500
- RN7: value 270 -> 470
- RN8, RN9: value 1800 -> 3300
- U10: value 74LS174 -> 74F574; footprint Package_DIP:DIP-16_W7.62mm_LongPads -> Package_DIP:DIP-20_W7.62mm_LongPads
- moved C24 25.4 mm to (101.6, 137.2)
- moved U8 5.08 mm to (99.1, 218.4)
- moved C26 4.07 mm to (63.5, 189.2)
- moved C30 3.81 mm to (92.7, 218.4)
- moved RN1 3.59 mm to (91.4, 189.2)
- moved U12 3.59 mm to (80.0, 189.2)
- moved U24 3.59 mm to (67.3, 189.2)
- moved C27 3.17 mm to (95.2, 189.2)
- moved U11 2.84 mm to (99.1, 189.2)
- moved C23 2.62 mm to (63.5, 147.3)
- moved U28 2.54 mm to (52.1, 147.3)
- moved U13 2.54 mm to (113.0, 218.4)
- moved U7 2.54 mm to (80.0, 218.2)
- moved C29 2.54 mm to (58.4, 221.0)
- moved U2 2.54 mm to (63.5, 221.0)
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- renumbered RN6 to RN1, RN1 to RN2, RN2 to RN3, RN3 to RN4, RN4 to RN5, RN11 to RN6
Connections:
- net /CPU/HL0 renamed Net-(U23-Pad19)
- net /CPU/HL1 renamed Net-(U23-Pad18)
- net /CPU/HL2 renamed Net-(U23-Pad17)
- net /CPU/HL3 renamed Net-(U23-Pad16)
- net /CPU/HL4 renamed Net-(U23-Pad15)
- net /CPU/HL5 renamed Net-(U23-Pad14)
- net /CPU/HL6 renamed Net-(U23-Pad13)
- net /CPU/HL7 renamed Net-(U23-Pad12)
- net tclk renamed /GPU/H0
- J6 pad 0: GNDA -> 0
- J6 pad 5: GNDA -> 0
- J6 pad 6: GNDA -> 0
- J6 pad 7: GNDA -> 0
- J6 pad 8: GNDA -> 0
- J6 pad 9: Net-(J6-Pad9) -> 1
- J7 pad 1: ~exle -> ~rom2
- J7 pad 22: 0 -> I15
- U1 pad 10: Net-(U1-Pad10) -> cclk
- U1 pad 9: cclk -> Net-(U1-Pad9)
- U10 pad 1: 1 -> 0
- U10 pad 10: ~pgoe -> 0
- U10 pad 11: Net-(U10-Pad11) -> dclk
- U10 pad 12: ~pcoe -> ~hloe
- U10 pad 13: Net-(U10-Pad13) -> ~alue
- U10 pad 14: Net-(U10-Pad14) -> ~pcoe
- U10 pad 15: ~alue -> ~pgoe
- U10 pad 16: 1 -> ~yoe
- U10 pad 2: Net-(U10-Pad2) -> ~inst
- U10 pad 3: ~inst -> ~gsync
- U10 pad 5: ~voe -> Net-(U10-Pad5)
- U10 pad 7: ~xoe -> Net-(U10-Pad7)
- U10 pad 8: 0 -> Net-(U10-Pad8)
- U10 pad 9: dclk -> Net-(U10-Pad9)
- U14 pad 13: ~hloe -> mv
- U23 pad 1: ~hloe -> 0
- U24 pad 15: ~alue -> ~hloe
- U25 pad 12: Net-(U25-Pad12) -> mode1
- U26 pad 1: ~xoe -> pclk1
- U27 pad 1: pclk1 -> ~yoe
- U3 pad 6: Net-(U1-Pad10) -> Net-(U1-Pad9)
- U35 pad 12: mode1 -> Net-(U35-Pad12)
- U38 pad 19: Net-(U1-Pad10) -> Net-(U1-Pad9)
- U41 pad 16: VDD -> 1
- U41 pad 7: VEE -> 0
- U41 pad 8: GNDA -> 0
- U5 pad 10: Net-(U10-Pad13) -> Net-(U10-Pad7)
- U5 pad 11: ~exle -> Net-(U10-Pad9)
- U5 pad 12: ~rom2 -> Net-(U10-Pad8)
- U5 pad 13: I15 -> mv
- U5 pad 6: Net-(U10-Pad6) -> Net-(U10-Pad5)
- U5 pad 8: Net-(U10-Pad11) -> Net-(U10-Pad6)
- U6 pad 8: ~hsync -> ~gsync
- U7 pad 6: Net-(U10-Pad13) -> Net-(U10-Pad7)
- U7 pad 7: Net-(U10-Pad14) -> Net-(U10-Pad8)
- U8 pad 13: Net-(U10-Pad2) -> Net-(U10-Pad19)
