File: eda/kicad/novasaur-io.sch (KiCad schematic (older format))
At the start: 72 parts, among them J1 POWER IN, J10 V H SYNC, J3 AUDIO OUT, J4 KEYBOARD, J5 SERIAL, J5 SPKR, J6 DISPLAY, J7 EXPANSION, J8 EXP OUT, J9 R G B, Q1 2N3904, Q2 2N3904, Q4 BS270, SW1 POWER, U1 74F86, U2 74F08, U38 74HCT4053, U39 MAX232, U4 74F32, U40 NJM4580, U41 MCP1827S, U6 74ALS139, U7 74ALS139

Commit message: update serial
Parts:
- removed Q1, Q2: 2N3904, Package_TO_SOT_THT:TO-92_HandSolder, symbol Transistor_BJT:2N3904
- removed R4: 1k, Resistor_THT:R_Axial_DIN0204_L3.6mm_D1.6mm_P7.62mm_Horizontal, symbol Device:R_US
- added D2, D4: BAT42, Diode_THT:D_DO-35_SOD27_P7.62mm_Horizontal, symbol Device:D_Schottky_ALT
- R3, R5: value 1k -> 10k
- R8: renamed from R9; value 100k -> 10k
- R9: renamed from R10; value 100k -> 10k
- renumbered D2 to D3, D3 to D5, R5 to R4, R6 to R5, R7 to R6, R8 to R7
Connections:
- net VCC: now also R5.1
- net VDD: now also J5.4
- net rts: now also D2.1 (K); no longer R5.2
- net tx: now also D3.1 (K); no longer D3.2 (A)
- net Ei0 renamed rx
- net Ei1 renamed cts
- net Ei2 renamed ps2clk
- net ps2clk: now also D3.2 (A), R5.2, D2.2 (A); no longer R3.2
- net Ei3 renamed ps2rx
- net ps2rx: now also R3.2, D4.2 (A)
- net T0 renamed F0
- net T1 renamed F1
- net T2 renamed F2
- net T3 renamed F3
- net T4 renamed F4
- net T5 renamed F5
- net T6 renamed F6
- net T7 renamed F7
- new net ps2tx: D4.1 (K)
- no-connect marks 12 -> 11
Other:
- moved on the sheet: C17, J10, J2, J7, J8, R2, R3, TP32
