File: eda/kicad/exp-proto/EXP.kicad_pcb (KiCad board)
At the start: 2 copper layers, 94 x 88.9 mm, 23 parts, among them J1 IN, J2 IN, J3 OUT, J4 OUT, J5 On, J6 On, J7 KEYPAD, J8 INTR, U1 74F138, U2 74F138, U3 74F574, U4 74F174, U5 74F244, U6 MCP1702-5002E

Commit message: add notes to schematic
Parts:
- J6: value On -> In
Changed lines of the file:
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@@
       (effects (font (size 1 1) (thickness 0.15)))
     )
-    (fp_text value "On" (at 1.27 20.11) (layer "F.Fab")
+    (fp_text value "In" (at 1.27 20.11) (layer "F.Fab")
       (effects (font (size 1 1) (thickness 0.15)))
     )
