File: cad/kicad/exp-proto/EXP.kicad_pcb (KiCad board)
At the start: 2 copper layers, 94 x 88.9 mm, 23 parts, among them J1 IN, J2 IN, J3 OUT, J4 OUT, J5 On, J6 In, J7 KEYPAD, J8 INTR, U1 74F138, U2 74F138, U3 74F574, U4 74F174, U5 74F244, U6 MCP1702-5002E

Commit message: update old C-reg labels
Connections:
- net C3 renamed C11
- D1 pad 2: C1 -> C9
- J2 pad 7: C1 -> C9
- J4 pad 5: C8 -> C0
- J4 pad 6: C9 -> C1
- J4 pad 7: C0 -> C8
- U1 pad 1: C8 -> C0
- U1 pad 2: C9 -> C1
- U1 pad 3: C0 -> C8
- U2 pad 1: C8 -> C0
- U2 pad 2: C9 -> C1
- U2 pad 3: C0 -> C8
Routing:
- net C9: track 63.4 -> 19.0 mm, vias 3 -> 1
- net C1: track 19.0 -> 63.4 mm, vias 1 -> 3
- net C8: track 59.9 -> 68.9 mm
- net C0: track 68.9 -> 59.9 mm
